Commit message: dim changed

File: irc_ros_ws/src/rover_base_description/urdf/rover_base_description.urdf.xacro (robot description, xacro)
@@ -8,6 +8,6 @@
   <xacro:property name="base_height" value="0.05" />
   <xacro:property name="wheel_mass" value="0.3" /> <!-- arbitrary value for wheel mass -->
-  <xacro:property name="wheel_len" value="0.020" />
-  <xacro:property name="wheel_radius" value="0.015" />
+  <xacro:property name="wheel_len" value="0.10" />
+  <xacro:property name="wheel_radius" value="0.10" />
   <xacro:property name="caster_wheel_mass" value="0.1" /> <!-- arbitrary value for caster wheel mass -->
   <xacro:property name="caster_wheel_radius" value="0.015" />
