Commit message: made changes in arm urdf and controls

File: irc_ros_ws/src/arm_description/urdf/arm.ros2_control.xacro (robot description, xacro)
@@ -4,5 +4,5 @@
         <hardware>
             <plugin>mock_components/GenericSystem</plugin>
-            <param name="calculate_dynamics">true</param>
+            <param name="calculate_dynamics">false</param>
             <!-- <plugin>arm_hardware/ArmHardwareInterface</plugin>
             <param name="joint1_motor_id">10</param>

File: irc_ros_ws/src/arm_description/urdf/arm.xacro (robot description, xacro)
@@ -4,5 +4,5 @@
 <xacro:include filename="$(find arm_description)/urdf/materials.xacro" />
 <xacro:include filename="$(find arm_description)/urdf/arm.trans" />
-<xacro:include filename="$(find arm_description)/urdf/arm.gazebo" />
+<!-- <xacro:include filename="$(find arm_description)/urdf/arm.gazebo" /> -->
 <xacro:include filename="$(find arm_description)/urdf/arm.ros2_control.xacro" />
 </robot>

File: irc_ros_ws/src/arm_description/urdf/arm_base.xacro (robot description, xacro)
@@ -3,7 +3,7 @@
 <link name="base_link">
   <inertial>
-    <origin xyz="-0.007360989774630262 0.025644899800482967 -0.0024952231420034905" rpy="0 0 0"/>
+    <origin xyz="-0.0010063158166902576 -0.0023179609946681447 0.0025047768579964246" rpy="0 0 0"/>
     <mass value="0.8402300230207919"/>
-    <inertia ixx="0.005301" iyy="0.003466" izz="0.008764" ixy="0.000207" iyz="-0.0" ixz="0.0"/>
+    <inertia ixx="0.005299" iyy="0.003467" izz="0.008764" ixy="0.000215" iyz="-0.0" ixz="0.0"/>
   </inertial>
   <visual>
@@ -23,10 +23,10 @@
 <link name="waist_1">
   <inertial>
-    <origin xyz="-0.0005513978901202954 0.009816058653192404 0.026001137569438594" rpy="0 0 0"/>
+    <origin xyz="-7.702444876018025e-05 0.009830969674369704 0.02300113756943942" rpy="0 0 0"/>
     <mass value="0.8480827984091125"/>
-    <inertia ixx="0.001216" iyy="0.00212" izz="0.002523" ixy="-5.1e-05" iyz="-8.3e-05" ixz="5e-06"/>
+    <inertia ixx="0.001213" iyy="0.002123" izz="0.002523" ixy="-7e-06" iyz="-8.3e-05" ixz="1e-06"/>
   </inertial>
   <visual>
-    <origin xyz="0.0 -0.0 -0.0" rpy="0 0 0"/>
+    <origin xyz="-0.00646 0.027932 -0.005" rpy="0 0 0"/>
     <geometry>
       <mesh filename="file://$(find arm_description)/meshes/waist_1.stl" scale="0.001 0.001 0.001"/>
@@ -35,5 +35,5 @@
   </visual>
   <collision>
-    <origin xyz="0.0 -0.0 -0.0" rpy="0 0 0"/>
+    <origin xyz="-0.00646 0.027932 -0.005" rpy="0 0 0"/>
     <geometry>
       <mesh filename="file://$(find arm_description)/meshes/waist_1.stl" scale="0.001 0.001 0.001"/>
@@ -43,10 +43,10 @@
 <link name="shoulder_1">
   <inertial>
-    <origin xyz="0.004641427187129456 -0.08259133662509736 0.2177413761989421" rpy="0 0 0"/>
+    <origin xyz="2.8948591498393662e-05 -0.004074156190009087 0.23288965236006828" rpy="0 0 0"/>
     <mass value="2.3356160941174426"/>
-    <inertia ixx="0.059469" iyy="0.054008" izz="0.008594" ixy="0.000308" iyz="0.018072" ixz="-0.001015"/>
+    <inertia ixx="0.059486" iyy="0.060319" izz="0.002265" ixy="-7e-06" iyz="-0.000522" ixz="5e-06"/>
   </inertial>
   <visual>
-    <origin xyz="-1e-06 -0.0 -0.0385" rpy="0 0 0"/>
+    <origin xyz="-0.006461 0.027932 -0.0405" rpy="0 0 0"/>
     <geometry>
       <mesh filename="file://$(find arm_description)/meshes/shoulder_1.stl" scale="0.001 0.001 0.001"/>
@@ -55,5 +55,5 @@
   </visual>
   <collision>
-    <origin xyz="-1e-06 -0.0 -0.0385" rpy="0 0 0"/>
+    <origin xyz="-0.006461 0.027932 -0.0405" rpy="0 0 0"/>
     <geometry>
       <mesh filename="file://$(find arm_description)/meshes/shoulder_1.stl" scale="0.001 0.001 0.001"/>
@@ -63,10 +63,10 @@
 <link name="forearm_1">
   <inertial>
-    <origin xyz="0.014992277113350418 -0.21413410482994938 0.06412032690918101" rpy="0 0 0"/>
+    <origin xyz="-0.0047246620557192965 0.22397119357725606 0.002083108957369073" rpy="0 0 0"/>
     <mass value="1.9893346240282717"/>
-    <inertia ixx="0.050093" iyy="0.008264" izz="0.049749" ixy="0.00364" iyz="0.013335" ixz="-0.001115"/>
+    <inertia ixx="0.050345" iyy="0.004096" izz="0.053666" ixy="0.001691" iyz="-0.000192" ixz="-1e-06"/>
   </inertial>
   <visual>
-    <origin xyz="-0.008568 0.152329 -0.461847" rpy="0 0 0"/>
+    <origin xyz="-0.006462 0.028078 -0.4905" rpy="0 0 0"/>
     <geometry>
       <mesh filename="file://$(find arm_description)/meshes/forearm_1.stl" scale="0.001 0.001 0.001"/>
@@ -75,5 +75,5 @@
   </visual>
   <collision>
-    <origin xyz="-0.008568 0.152329 -0.461847" rpy="0 0 0"/>
+    <origin xyz="-0.006462 0.028078 -0.4905" rpy="0 0 0"/>
     <geometry>
       <mesh filename="file://$(find arm_description)/meshes/forearm_1.stl" scale="0.001 0.001 0.001"/>
@@ -83,10 +83,10 @@
 <link name="wrist_1_1">
   <inertial>
-    <origin xyz="-0.0654930878436422 -0.005004021827981986 0.002033641911817874" rpy="0 0 0"/>
+    <origin xyz="-0.06568494427723634 0.001506419448577545 -0.0013244463243618498" rpy="0 0 0"/>
     <mass value="1.139710997448956"/>
-    <inertia ixx="0.000446" iyy="0.002949" izz="0.003038" ixy="4.1e-05" iyz="-3.5e-05" ixz="1.6e-05"/>
+    <inertia ixx="0.000461" iyy="0.002977" izz="0.002995" ixy="-0.00018" iyz="-6.2e-05" ixz="-8.6e-05"/>
   </inertial>
   <visual>
-    <origin xyz="-0.032821 0.58353 -0.588248" rpy="0 0 0"/>
+    <origin xyz="-0.002883 -0.421905 -0.492176" rpy="0 0 0"/>
     <geometry>
       <mesh filename="file://$(find arm_description)/meshes/wrist_1_1.stl" scale="0.001 0.001 0.001"/>
@@ -95,5 +95,5 @@
   </visual>
   <collision>
-    <origin xyz="-0.032821 0.58353 -0.588248" rpy="0 0 0"/>
+    <origin xyz="-0.002883 -0.421905 -0.492176" rpy="0 0 0"/>
     <geometry>
       <mesh filename="file://$(find arm_description)/meshes/wrist_1_1.stl" scale="0.001 0.001 0.001"/>
@@ -103,10 +103,10 @@
 <link name="wrist_2_1">
   <inertial>
-    <origin xyz="0.0008772605587413218 -0.015596392296797101 0.007267252182415751" rpy="0 0 0"/>
+    <origin xyz="-0.0001378319350452636 0.017225594312011316 -0.00031580323993046777" rpy="0 0 0"/>
     <mass value="0.1496451428941353"/>
-    <inertia ixx="3.6e-05" iyy="6.3e-05" izz="5.3e-05" ixy="-1e-06" iyz="-6e-06" ixz="1e-06"/>
+    <inertia ixx="3.6e-05" iyy="6.6e-05" izz="5e-05" ixy="-0.0" iyz="-0.0" ixz="-1e-06"/>
   </inertial>
   <visual>
-    <origin xyz="-0.034348 0.610682 -0.600914" rpy="0 0 0"/>
+    <origin xyz="-0.002645 -0.451898 -0.491615" rpy="0 0 0"/>
     <geometry>
       <mesh filename="file://$(find arm_description)/meshes/wrist_2_1.stl" scale="0.001 0.001 0.001"/>
@@ -115,5 +115,5 @@
   </visual>
   <collision>
-    <origin xyz="-0.034348 0.610682 -0.600914" rpy="0 0 0"/>
+    <origin xyz="-0.002645 -0.451898 -0.491615" rpy="0 0 0"/>
     <geometry>
       <mesh filename="file://$(find arm_description)/meshes/wrist_2_1.stl" scale="0.001 0.001 0.001"/>
@@ -121,38 +121,33 @@
   </collision>
 </link>
-<joint name="turret_joint" type="revolute">
-  <origin xyz="0.0 0.0 0.0" rpy="0 0 0"/>
+<joint name="turret_joint" type="continuous">
+  <origin xyz="0.00646 -0.027932 0.005" rpy="0 0 0"/>
   <parent link="base_link"/>
   <child link="waist_1"/>
   <axis xyz="0.0 0.0 1.0"/>
-  <limit upper="${pi}" lower="${-pi}" effort="100" velocity="100"/>
 </joint>
-<joint name="shoulder_joint" type="revolute">
-  <origin xyz="1e-06 0.0 0.0385" rpy="0 0 0"/>
+<joint name="shoulder_joint" type="continuous">
+  <origin xyz="1e-06 0.0 0.0355" rpy="0 0 0"/>
   <parent link="waist_1"/>
   <child link="shoulder_1"/>
-  <axis xyz="0.998422 0.056156 -0.0"/>
-  <limit upper="1.919862" lower="${-pi}" effort="100" velocity="100"/>
+  <axis xyz="0.999968 0.007954 0.0"/>
 </joint>
-<joint name="elbow_joint" type="revolute">
-  <origin xyz="0.008567 -0.152329 0.423347" rpy="0.652 0 0"/>
+<joint name="elbow_joint" type="continuous">
+  <origin xyz="1e-06 -0.000146 0.45" rpy="0 0 0"/>
   <parent link="shoulder_1"/>
   <child link="forearm_1"/>
-  <axis xyz="-1.0 0.0 0.0"/>
-  <limit upper="0.6" lower="0.0" effort="100" velocity="100"/>
+  <axis xyz="-0.999968 -0.007954 -0.0"/>
 </joint>
-<joint name="wrist_pitch" type="revolute">
-  <origin xyz="0.024253 -0.431201 0.126401" rpy="0 0 0"/>
+<joint name="wrist_pitch" type="continuous">
+  <origin xyz="-0.003579 0.449983 0.001676" rpy="0 0 0"/>
   <parent link="forearm_1"/>
   <child link="wrist_1_1"/>
-  <axis xyz="0.998422 0.056156 -0.0"/>
-  <limit upper="${pi / 2}" lower="-${pi / 2}" effort="100" velocity="100"/>
+  <axis xyz="-0.999968 -0.007954 -0.0"/>
 </joint>
-<joint name="wrist_roll" type="revolute">
-  <origin xyz="0.001527 -0.027152 0.012666" rpy="0 0 0"/>
+<joint name="wrist_roll" type="continuous">
+  <origin xyz="-0.000238 0.029993 -0.000561" rpy="0 0 0"/>
   <parent link="wrist_1_1"/>
   <child link="wrist_2_1"/>
-  <axis xyz="0.050906 -0.905077 0.422189"/>
-  <limit upper="${pi}" lower="${-pi}" effort="100" velocity="100"/>
+  <axis xyz="-0.007952 0.999793 -0.018724"/>
 </joint>
 </robot>

Commit message: arm controller to joint cmd

File: irc_ros_ws/src/arm_description/urdf/arm.ros2_control.xacro (robot description, xacro)
@@ -11,8 +11,8 @@
             <param name="pid_o">50</param>
         </hardware>
-        <joint name="turret_joint">
+        <joint name="elbow_joint">
             <command_interface name="position" />
             <state_interface name="position" />
-            <state_interface name="velocity" />
+            <!-- <state_interface name="velocity" /> -->
             <param name="encoder_counts_per_rev">8192</param>
         </joint>
@@ -20,11 +20,11 @@
             <command_interface name="position" />
             <state_interface name="position" />
-            <state_interface name="velocity" />
+            <!-- <state_interface name="velocity" /> -->
             <param name="encoder_counts_per_rev">8192</param>
         </joint>
-        <joint name="elbow_joint">
+        <joint name="turret_joint">
             <command_interface name="position" />
             <state_interface name="position" />
-            <state_interface name="velocity" />
+            <!-- <state_interface name="velocity" /> -->
             <param name="encoder_counts_per_rev">8192</param>
         </joint>
@@ -32,5 +32,5 @@
             <command_interface name="position" />
             <state_interface name="position" />
-            <state_interface name="velocity" />
+            <!-- <state_interface name="velocity" /> -->
             <param name="encoder_counts_per_rev">8192</param>
         </joint>
@@ -38,5 +38,5 @@
             <command_interface name="position" />
             <state_interface name="position" />
-            <state_interface name="velocity" />
+            <!-- <state_interface name="velocity" /> -->
             <param name="encoder_counts_per_rev">8192</param>
         </joint>

Commit message: made urdf correct

File: irc_ros_ws/src/arm_description/urdf/arm.ros2_control.xacro (robot description, xacro)
@@ -15,4 +15,5 @@
             <command_interface name="velocity" />
             <state_interface name="position" />
+            <state_interface name="velocity" />
             <param name="encoder_counts_per_rev">8192</param>
         </joint>
@@ -21,4 +22,5 @@
             <command_interface name="velocity" />
             <state_interface name="position" />
+            <state_interface name="velocity" />
             <param name="encoder_counts_per_rev">8192</param>
         </joint>
@@ -27,4 +29,5 @@
             <command_interface name="velocity" />
             <state_interface name="position" />
+            <state_interface name="velocity" />
             <param name="encoder_counts_per_rev">8192</param>
         </joint>
@@ -33,4 +36,5 @@
             <command_interface name="velocity" />
             <state_interface name="position" />
+            <state_interface name="velocity" />
             <param name="encoder_counts_per_rev">8192</param>
         </joint>
@@ -39,4 +43,5 @@
             <command_interface name="velocity" />
             <state_interface name="position" />
+            <state_interface name="velocity" />
             <param name="encoder_counts_per_rev">8192</param>
         </joint>

File: irc_ros_ws/src/arm_description/urdf/arm_base.xacro (robot description, xacro)
@@ -129,12 +129,12 @@
 </joint>
 <joint name="shoulder_joint" type="revolute">
-  <origin xyz="1e-06 0.0 0.0355" rpy="0 0 0"/>
+  <origin xyz="1e-06 0.0 0.0355" rpy="-0.289729 0 0"/>
   <parent link="waist_1"/>
   <child link="shoulder_1"/>
-  <axis xyz="0.999968 0.007954 0.0"/>
+  <axis xyz="-0.999968 -0.007954 0.0"/>
   <limit lower="${-pi/2}" upper="-0.17" effort="0.0" velocity="0.0"/>
 </joint>
 <joint name="elbow_joint" type="revolute">
-  <origin xyz="1e-06 -0.000146 0.45" rpy="0 0 0"/>
+  <origin xyz="1e-06 -0.000146 0.45" rpy="-0.350289 0 0"/>
   <parent link="shoulder_1"/>
   <child link="forearm_1"/>
@@ -143,5 +143,5 @@
 </joint>
 <joint name="wrist_pitch" type="revolute">
-  <origin xyz="-0.003579 0.449983 0.001676" rpy="0 0 0"/>
+  <origin xyz="-0.003579 0.449983 0.001676" rpy="0.640018 0 0"/>
   <parent link="forearm_1"/>
   <child link="wrist_1_1"/>

Commit message: changes

File: irc_ros_ws/src/arm_description/urdf/arm.ros2_control.xacro (robot description, xacro)
@@ -3,67 +3,37 @@
     <ros2_control name="Arm" type="system">
         <hardware>
-            <!-- <plugin>mock_components/GenericSystem</plugin>
-            <param name="calculate_dynamics">false</param> -->
-            <plugin>arm/ArmHardware</plugin>
+            <plugin>mock_components/GenericSystem</plugin>
+            <param name="calculate_dynamics">false</param>
+            <!-- <plugin>arm/ArmHardware</plugin> -->
         </hardware>
         <joint name="elbow_joint">
-            <!-- <command_interface name="position" /> -->
-            <command_interface name="velocity" />
+            <command_interface name="position" />
             <state_interface name="position" />
-            <state_interface name="velocity" />
-            <param name="encoder_counts_per_rev">8192</param>
-            <param name="pid_p">100</param>
-            <param name="pid_d">0</param>
-            <param name="pid_i">0.000</param>
-            <param name="max_pwm">130</param>
-            <param name="min_pwm">-130</param>
+            <!-- <state_interface name="velocity" /> -->
         </joint>
         <joint name="shoulder_joint">
-            <!-- <command_interface name="position" /> -->
-            <command_interface name="velocity" />
+            <command_interface name="position" />
             <state_interface name="position" />
-            <state_interface name="velocity" />
-            <param name="encoder_counts_per_rev">8192</param>
-            <param name="pid_p">200</param>
-            <param name="pid_d">0</param>
-            <param name="pid_i">0.000</param>
-            <param name="max_pwm">254</param>
-            <param name="min_pwm">-254</param>
+            <!-- <state_interface name="velocity" /> -->
         </joint>
         <joint name="turret_joint">
-            <!-- <command_interface name="position" /> -->
-            <command_interface name="velocity" />
+            <command_interface name="position" />
             <state_interface name="position" />
-            <state_interface name="velocity" />
-            <param name="encoder_counts_per_rev">460000</param>
-            <param name="pid_p">30</param>
-            <param name="pid_d">0</param>
-            <param name="pid_i">0.000</param>
-            <param name="max_pwm">70.0</param>
-            <param name="min_pwm">-70.0</param>
+            <!-- <state_interface name="velocity" /> -->
         </joint>
         <joint name="wrist_pitch">
-            <!-- <command_interface name="position" /> -->
-            <command_interface name="velocity" />
+            <command_interface name="position" />
             <state_interface name="position" />
-            <state_interface name="velocity" />
-            <param name="encoder_counts_per_rev">8192</param>
-            <param name="pid_p">40</param>
-            <param name="pid_d">0</param>
-            <param name="pid_i">0.000</param>
-            <param name="max_pwm">40.0</param>
-            <param name="min_pwm">-40.0</param>
+            <!-- <state_interface name="velocity" /> -->
         </joint>
         <joint name="wrist_roll">
-            <!-- <command_interface name="position" /> -->
-            <command_interface name="velocity" />
+            <command_interface name="position" />
             <state_interface name="position" />
-            <state_interface name="velocity" />
-            <param name="encoder_counts_per_rev">8192</param>
-            <param name="pid_p">1.0</param>
-            <param name="pid_d">5.0</param>
-            <param name="pid_i">0.000</param>
-            <param name="max_pwm">40.0</param>
-            <param name="min_pwm">-40.0</param>
+            <!-- <state_interface name="velocity" /> -->
+        </joint>
+        <joint name="gripper_motor_joint">
+            <command_interface name="position" />
+            <state_interface name="position" />
+            <!-- <state_interface name="velocity" /> -->
         </joint>
     </ros2_control>

File: irc_ros_ws/src/arm_description/urdf/arm_base.xacro (robot description, xacro)
@@ -121,4 +121,24 @@
   </collision>
 </link>
+<link name="gripper_motor">
+  <inertial>
+    <origin xyz="0.0 0.0 0.0" rpy="0 0 0"/>
+    <mass value="1.0"/>
+    <inertia ixx="3.5625e-05" iyy="3.5625e-05" izz="1.125e-05" ixy="0.0" iyz="0.0" ixz="0.0"/>
+  </inertial>
+  <visual>
+    <origin xyz="0.0 0.0 0.0" rpy="0 1.57 0"/>
+    <geometry>
+      <cylinder radius="0.015" length="0.06"/>
+    </geometry>
+    <material name="silver"/>
+  </visual>
+  <collision>
+    <origin xyz="0.0 0.0 0.0" rpy="0 3.14 0"/>
+    <geometry>
+      <cylinder radius="0.015" length="0.06"/>
+    </geometry>
+  </collision>
+</link>
 <joint name="turret_joint" type="revolute">
   <origin xyz="0.00646 -0.027932 0.005" rpy="0 0 0"/>
@@ -129,5 +149,5 @@
 </joint>
 <joint name="shoulder_joint" type="revolute">
-  <origin xyz="1e-06 0.0 0.0355" rpy="-0.289729 0 0"/>
+  <origin xyz="1e-06 0.0 0.0355" rpy="0 0 0"/>
   <parent link="waist_1"/>
   <child link="shoulder_1"/>
@@ -136,5 +156,5 @@
 </joint>
 <joint name="elbow_joint" type="revolute">
-  <origin xyz="1e-06 -0.000146 0.45" rpy="-0.350289 0 0"/>
+  <origin xyz="1e-06 -0.000146 0.45" rpy="0 0 0"/>
   <parent link="shoulder_1"/>
   <child link="forearm_1"/>
@@ -143,5 +163,5 @@
 </joint>
 <joint name="wrist_pitch" type="revolute">
-  <origin xyz="-0.003579 0.449983 0.001676" rpy="0.640018 0 0"/>
+  <origin xyz="-0.003579 0.449983 0.001676" rpy="0 0 0"/>
   <parent link="forearm_1"/>
   <child link="wrist_1_1"/>
@@ -156,3 +176,9 @@
   <limit lower="${-pi/2}" upper="${pi/2}" effort="0.0" velocity="0.0"/>
 </joint>
+<joint name="gripper_motor_joint" type="continuous">
+  <origin xyz="0.0 0.029993 -0.000561" rpy="0 0 0"/>
+  <parent link="wrist_2_1"/>
+  <child link="gripper_motor"/>
+  <axis xyz="1 0 0"/>
+</joint>
 </robot>

File: irc_ros_ws/src/irc_rover_description/urdf/kartikeya.xacro (robot description, xacro)
@@ -337,5 +337,5 @@
   <parent link="waist_1"/>
   <child link="shoulder_1"/>
-  <axis xyz="1.0 -0.000773 0.0"/>
+  <axis xyz="-1.0 -0.000773 0.0"/>
 </joint>
 <joint name="elbow_joint" type="continuous">

File: irc_ros_ws/src/irc_rover_description/urdf/kartikeya_arm.ros2_control.xacro (robot description, xacro)
@@ -13,7 +13,7 @@
             <state_interface name="velocity" />
             <param name="encoder_counts_per_rev">8192</param>
-            <param name="pid_p">200</param>
+            <param name="pid_p">1000</param>
             <param name="pid_d">0</param>
-            <param name="pid_i">0.000</param>
+            <param name="pid_i">1</param>
             <param name="max_pwm">250</param>
             <param name="min_pwm">-250</param>
@@ -25,7 +25,7 @@
             <state_interface name="velocity" />
             <param name="encoder_counts_per_rev">8192</param>
-            <param name="pid_p">100</param>
+            <param name="pid_p">150</param>
             <param name="pid_d">0</param>
-            <param name="pid_i">0.000</param>
+            <param name="pid_i">0.1</param>
             <param name="max_pwm">120</param>
             <param name="min_pwm">-120</param>
@@ -50,6 +50,6 @@
             <param name="encoder_counts_per_rev">8192</param>
             <param name="pid_p">15</param>
-            <param name="pid_d">0</param>
-            <param name="pid_i">0.000</param>
+            <param name="pid_d">10</param>
+            <param name="pid_i">0.0003</param>
             <param name="max_pwm">30.0</param>
             <param name="min_pwm">-30.0</param>
